File: kicad/psu-board/psu-board.kicad_pcb (KiCad board)
At the start: 4 copper layers, 66.7 x 38.1 mm, 39 parts, among them J1 Vin, J10 GND, J2 GND, J3 Vout+, J4 GND, J5 Vout-

Commit message: more data
Parts:
- removed J10: GND, Connector_Wire:SolderWire-0.5sqmm_1x01_D0.9mm_OD2.3mm
- removed J3: Vout+, Connector_Wire:SolderWire-0.5sqmm_1x01_D0.9mm_OD2.3mm
- added D5: GREEN, LED_THT:LED_D5.0mm, B.Cu at (139.7, 101.6)
- added J6: Vout+, Connector_Wire:SolderWire-0.5sqmm_1x01_D0.9mm_OD2.3mm, F.Cu at (160.0, 118.1)
- added R10: 3k, Resistor_SMD:R_0805_2012Metric, F.Cu at (149.8, 107.1)
- added R11: 3k, Resistor_SMD:R_0805_2012Metric, F.Cu at (156.2, 121.0)
- added R5: 10k, Resistor_SMD:R_0805_2012Metric, F.Cu at (146.1, 101.6)
- added R6: 0, Resistor_SMD:R_0805_2012Metric, F.Cu at (123.0, 98.7)
- added R7: 0, Resistor_SMD:R_0805_2012Metric, F.Cu at (123.0, 100.9)
- C1: value 22uF -> 200uF; footprint Capacitor_SMD:C_1206_3216Metric -> Capacitor_THT:CP_Radial_D10.0mm_P5.00mm; moved to B.Cu
- C12: value 200uF -> 10n; footprint Capacitor_THT:CP_Radial_D10.0mm_P5.00mm -> Capacitor_SMD:C_1206_3216Metric
- C13: value 10p -> 200uF; footprint Capacitor_SMD:C_1206_3216Metric -> Capacitor_THT:CP_Radial_D10.0mm_P5.00mm; moved to B.Cu
- C14: value 10n -> 200uF; footprint Capacitor_SMD:C_1206_3216Metric -> Capacitor_THT:CP_Radial_D10.0mm_P5.00mm; moved to B.Cu
- C15: value 10n -> 10p
- C2: value 200uF -> 2uF; footprint Capacitor_THT:CP_Radial_D10.0mm_P5.00mm -> Capacitor_SMD:C_1206_3216Metric; moved to F.Cu
- C3: value 2uF -> 22uF
- C5: value 22uF -> 10n
- C8: moved to F.Cu
- C9: value 200uF -> 22uF; footprint Capacitor_THT:CP_Radial_D10.0mm_P5.00mm -> Capacitor_SMD:C_1206_3216Metric; moved to F.Cu
- D1: value STPS340 -> 1N5404; footprint Diode_SMD:D_SMB -> Diode_THT:D_DO-41_SOD81_P3.81mm_Vertical_AnodeUp
- D2: value STPS340 -> 7.5V; footprint Diode_SMD:D_SMB -> Diode_SMD:D_MiniMELF
- D3: value 8.2V -> STPS340; footprint Diode_SMD:D_MiniMELF -> Diode_SMD:D_SMB
- D4: value 1N5404 -> STPS340; footprint Diode_THT:D_DO-41_SOD81_P10.16mm_Horizontal -> Diode_SMD:D_SMB; moved to F.Cu
- L2, L3: moved to B.Cu
- R2: value 10k -> 1k
- R3: value 1k -> 10k
- moved H1 89.3 mm to (103.8, 99.1)
- moved H2 89.3 mm to (162.8, 99.1)
- moved H4 89.3 mm to (103.8, 129.5)
- moved H3 89.3 mm to (162.8, 129.5)
- moved C14 46.1 mm to (156.2, 125.7), turned to 135 degrees
- moved L2 41.0 mm to (147.3, 130.8), turned to 90 degrees
- moved L3 33.7 mm to (147.3, 115.6), turned to 90 degrees
- moved C12 32.8 mm to (144.8, 114.3), turned to 90 degrees
- moved R2 32.8 mm to (116.7, 100.9), turned to 180 degrees
- moved RV1 29.0 mm to (118.0, 99.7)
- moved D1 28.2 mm to (112.4, 107.6), turned to 90 degrees
- moved R3 27.3 mm to (135.9, 100.3), turned to 0 degrees
- moved C1 25.1 mm to (120.7, 110.3), turned to 90 degrees
- moved D4 24.9 mm to (130.8, 130.8), turned to 180 degrees
- moved C3 24.6 mm to (131.9, 123.7), turned to 0 degrees
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Connections:
- C1 pad 1: Net-(C1-Pad1) -> /1
- C10 pad 1: Net-(C1-Pad1) -> /pos
- C11 pad 1: Net-(C1-Pad1) -> /3
- C12 pad 1: +VOUT -> /3
- C13 pad 1: FB -> GND
- C13 pad 2: +VOUT -> -VOUT
- C14 pad 1: Net-(C1-Pad1) -> +VOUT
- C15 pad 1: /3 -> FB
- C15 pad 2: GND -> +VOUT
- C3 pad 1: /1 -> /5
- C3 pad 2: GND -> /4
- C4 pad 1: /5 -> /6
- C4 pad 2: /4 -> /5
- C5 pad 1: /6 -> /pos
- C5 pad 2: /5 -> GND
- C6 pad 1: GND -> /pos
- C7 pad 2: GND -> /3
- C8 pad 1: /3 -> /pos
- C9 pad 2: GND -> /3
- D1 pad 1: GND -> /1
- D1 pad 2: /4 -> GND
- D2 pad 1: Net-(C1-Pad1) -> /1
- D2 pad 2: /5 -> Net-(D2-Pad2)
- D3 pad 1: /1 -> GND
- D3 pad 2: Net-(D3-Pad2) -> /4
- D4 pad 1: /1 -> /pos
- D4 pad 2: GND -> /5
- L1 pad 3: GND -> /3
- L2 pad 1: Net-(C1-Pad1) -> /pos
- R1 pad 1: GND -> Net-(D2-Pad2)
- R1 pad 2: FB -> GND
- R2 pad 1: FB -> Net-(RV1-Pad1)
- R2 pad 2: +VOUT -> FB
- R3 pad 1: GND -> FB
- R3 pad 2: FB -> +VOUT
- R4 pad 1: Net-(D3-Pad2) -> Net-(RV1-Pad1)
- R4 pad 2: GND -> FB
- RV1 pad 1: GND -> Net-(RV1-Pad1)
- VR1 pad 2: Net-(D3-Pad2) -> Net-(D2-Pad2)
Routing:
- net +VOUT: track 7.00 -> 75.0 mm
- net -VOUT: track 7.99 -> 71.9 mm, vias 0 -> 2
- net Net-(C1-Pad1): track 24.7 -> 0.00 mm
- net GND: track 219.5 -> 197.2 mm, vias 2 -> 4
- net Net-(D3-Pad2): track 21.7 -> 0.00 mm
- net /6: track 12.4 -> 32.2 mm
- net FB: track 40.4 -> 59.9 mm, vias 0 -> 2
- net /pos: track 0.00 -> 16.2 mm
- net /4: track 12.4 -> 28.2 mm, vias 0 -> 2
- net /3: track 0.00 -> 15.0 mm
- net /1: track 39.5 -> 25.0 mm
- net /5: track 19.8 -> 11.3 mm
- net Net-(D2-Pad2): track 0.00 -> 7.37 mm
- net Net-(RV1-Pad1): track 0.00 -> 6.79 mm
- net Net-(D5-Pad2): track 0.00 -> 2.90 mm
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Other:
- board text added: "A"
- board text added: "B"
- board text added: "C"
- board text added: "D"
