File: kicad/psu-board/psu-board.kicad_sch (KiCad schematic)
At the start: 39 parts, among them J1 Vin, J10 GND, J2 GND, J3 Vout+, J4 GND, J5 Vout-

Commit message: more data
Parts:
- removed J10: GND, Connector_Wire:SolderWire-0.5sqmm_1x01_D0.9mm_OD2.3mm, symbol Connector:Conn_01x01_Female
- added D5: GREEN, LED_THT:LED_D5.0mm, symbol Diode:1N4001
- added R10, R11: 3k, Resistor_SMD:R_0805_2012Metric, symbol Device:R_US
- added R5: 10k, Resistor_SMD:R_0805_2012Metric, symbol Device:R_US
- added R6, R7: 0, Resistor_SMD:R_0805_2012Metric, symbol Device:R_US
- added R8, R9: 1k, Resistor_SMD:R_0805_2012Metric, symbol Device:R_US
- D1: renamed from D4; footprint Diode_THT:D_DO-41_SOD81_P10.16mm_Horizontal -> Diode_THT:D_DO-41_SOD81_P3.81mm_Vertical_AnodeUp
- D2: renamed from D3; value 8.2V -> 7.5V
- renumbered C2 to C1, C11 to C10, C8 to C11, C15 to C12, C9 to C13, C12 to C14, C13 to C15, C3 to C2, C4 to C3, C5 to C4, C14 to C5, C1 to C6, C6 to C7, C10 to C8, C7 to C9, D1 to D3, D2 to D4, J3 to J6, R4 to R1, R1 to R2, R2 to R3, R3 to R4
Connections:
- net +VOUT: now also D5.1 (K), R11.1; no longer C13.1
- net -VOUT: now also R10.1, R6.2, R8.1, R9.1; no longer R2.1, R4.1, RV1.1
- net FB: now also R8.2, R9.2
- net GND: now also C13.1, R10.2, R11.2, R5.2, R7.2
- net pos: now reaches C10.1, C5.1, C6.1, C8.1, D4.1 (K), L2.1
- new net: R2.1, R4.1, R6.1, R7.1, RV1.1
- new net: D5.2 (A), R5.1
- no-connect marks 2 -> 1
Other:
- note added: "+15V, 150mA"
- note added: "-15V, 150mA"
- note removed: "+17V, 200mA"
- note removed: "-17V, 200mA"
- moved on the sheet: C1, C10, C11, C12, C13, C14, C15, C2, C3, C4, C5, C6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
